Commit message: 完成重定位功能，但2d栅格图模糊

File: src/elderbot_description/urdf/elderbot_properties.urdf.xacro (robot description, xacro)
@@ -19,5 +19,5 @@
   <!-- Laser (RPLidar C1): mounted at front, 16cm from center, 15cm above ground -->
   <xacro:property name="laser_pose">
-    <origin xyz="0.16 0 0.15" rpy="0 0 3.14159265" />
+    <origin xyz="0.16 0 0.85" rpy="0 0 3.14159265" />
   </xacro:property>
   <!-- Depth sensor (Orbbec Gemini 335): at x=0.16m, z=0.42m -->
